File: Mainboard/PikaPC_Mainboard.kicad_sch (KiCad schematic)
At the start: 88 parts, among them J1 Conn_02x08_Odd_Even, J10 Conn_01x08, J11 Conn_01x08, J12 Conn_01x08, J13 Conn_01x08, J14 Conn_01x08, J15 Conn_01x08, J16 Conn_01x08, J17 Conn_01x08, J18 Conn_01x10, J19 Conn_02x05_Odd_Even, J5 DIN41612_03x32_C_Split, J6 Mini-DIN-6, J7 Mini-DIN-6, J8 Conn_01x06, J9 Conn_01x08, SW1 SW_Push_DPDT, SW2 SW_Push, U1 PPC403GA, U10 74LS07, U11 86C325, U12 GD75232N, U13 74LVC125, U14 MCP120-315GI/TO, U15 AS6C4008-55PCN, U16 AS6C4008-55PCN, U17 ATF1504, U18 T224162B, U19 T224162B, U2 SN74LVC245A, U20 T224162B, U21 T224162B, U22 74LVC125, U3 SST39VF010, U4 SN74LVC245A, U5 SN74LVC245A, U6 SN74LVC245A, U7 8042 PS/2, U8 ATF22V10C, U9 74LS04, Y1 25M, Y2 7M3728, Y3 14M31818

Commit message: New peripheral bus
- additional bus transceivers for byte lane steering to VLB
- replace 22V10 with 1504 for peripheral bus control logic
Parts:
- removed J8: Conn_01x06, Connector_PinHeader_2.54mm:PinHeader_1x06_P2.54mm_Vertical, symbol Connector_Generic:Conn_01x06
- removed R4, R5, R8: 1k, Resistor_THT:R_Axial_DIN0204_L3.6mm_D1.6mm_P7.62mm_Horizontal, symbol Device:R_Small_US
- removed U22: 74LVC125, Package_DIP:DIP-14_W7.62mm_Socket, symbol 74xx:74LVC125
- removed U8: ATF22V10C, Package_DIP:DIP-24_W7.62mm_Socket, symbol Logic_Programmable:PAL20RS10
- added U22, U23, U8: SN74LVC245A, Package_DIP:DIP-20_W7.62mm_Socket, symbol 74xx:74LS245
Connections:
- net SDCS is gone; now on net ~{CS5}: U17.37 (IO53)
- net SDMISO is gone; now on net ~{CS3}: U17.41 (IO64)
- net SDMOSI is gone; now on net ~{CS2}: U17.40 (IO62)
- net SDSCK is gone; now on net ~{CS7}: U17.39 (IO57)
- net ~{VID-SRDYn} is gone; now on net ~{VID-SRDY}: RN4.8 (R7), U11.23 (~{SRDY}), U13.1
- net +3.3V: now also U22.20 (VCC), U23.20 (VCC), U8.20 (VCC); no longer U13.5
- net A0/~{WBE0}: now also U17.31 (IO46)
- net A1/~{WBE1}: now also U17.28 (IO40)
- net A23: now also U17.26 (IO36); no longer U11.8 (SM/~{IO})
- net D24: now also U22.18 (B0), U23.18 (B0), U8.18 (B0)
- net D25: now also U22.17 (B1), U23.17 (B1), U8.17 (B1)
- net D26: now also U22.16 (B2), U23.16 (B2), U8.16 (B2)
- net D27: now also U22.15 (B3), U23.15 (B3), U8.15 (B3)
- net D28: now also U22.14 (B4), U23.14 (B4), U8.14 (B4)
- net D29: now also U22.13 (B5), U23.13 (B5), U8.13 (B5)
- net D30: now also U22.12 (B6), U23.12 (B6), U8.12 (B6)
- net D31: now also U22.11 (B7), U23.11 (B7), U8.11 (B7)
- net GND: now also U22.10 (GND), U23.10 (GND), U8.10 (GND)
- net INT1: no longer U17.17 (IO24)
- net Ready: no longer U13.6
- net R/~{W}: now also U22.1 (A->B), U23.1 (A->B), U8.1 (A->B); no longer U17.11 (IO3)
- net SysClk-5v: now also U11.194 (SCLK); no longer U9.13
- net VID-SAUP1: now also U17.19 (IO20)
- net VID-SAUP2: now also U17.20 (IO19)
- net ~{CS4}: now also U17.36 (IO52); no longer U17.9 (IO4)
- net ~{CS6}: now also U17.34 (IO51)
- net ~{OE}: now also U17.33 (IO49)
- net ~{VID-ADS}: now also U17.4 (IO16)
- net ~{VID-RDYIN}: now also U17.12 (IO1)
- net ~{VID-SBE0}: now also U17.17 (IO24)
- net ~{VID-SBE1}: now also U17.14 (IO30)
- net ~{VID-SBE2}: now also U17.18 (IO21)
- net ~{VID-SBE3}: now also U17.16 (IO25)
- net ~{WBE2}: now also U17.27 (IO37)
- net ~{WBE3}: now also U17.29 (IO41)
- net PB-TMS: now reaches U17.13 (TMS/IO32)
- net ~{VID-SRDY}: now reaches U17.25 (IO35)
- net PB-TCK: now reaches U17.32 (TCK/IO48)
- net PB-TDO: now reaches U17.38 (TDO/IO56)
- net PB-TDI: now reaches U17.7 (TDI/IO8)
- net PD0 renamed VD24
- net VD24: now also U23.2 (A0)
- net PD1 renamed VD25
- net VD25: now also U23.3 (A1)
- net PD10 renamed VD18
- net VD18: now also U22.4 (A2)
- net PD11 renamed VD19
- net VD19: now also U22.5 (A3)
- net PD12 renamed VD20
- net VD20: now also U22.6 (A4)
- net PD13 renamed VD21
- net VD21: now also U22.7 (A5)
- net PD14 renamed VD22
- net VD22: now also U22.8 (A6)
- net PD15 renamed VD23
- net VD23: now also U22.9 (A7)
- net PD16 renamed VD8
- net VD8: now also U8.2 (A0)
- net PD17 renamed VD9
- net VD9: now also U8.3 (A1)
- net PD18 renamed VD10
- net VD10: now also U8.4 (A2)
- net PD19 renamed VD11
- net VD11: now also U8.5 (A3)
- net PD2 renamed VD26
- net VD26: now also U23.4 (A2)
- net PD20 renamed VD12
- net VD12: now also U8.6 (A4)
- net PD21 renamed VD13
- net VD13: now also U8.7 (A5)
- net PD22 renamed VD14
- net VD14: now also U8.8 (A6)
- net PD23 renamed VD15
- net VD15: now also U8.9 (A7)
- net PD24 renamed VD0
- net VD0: no longer U17.8 (IO5)
- net PD25 renamed VD1
- net VD1: no longer U17.6 (IO11)
- net PD26 renamed VD2
- net VD2: no longer U17.5 (IO14)
- net PD27 renamed VD3
- net VD3: no longer U17.4 (IO16)
- net PD28 renamed VD4
- net VD4: no longer U17.21 (IO17)
- net PD29 renamed VD5
- net VD5: no longer U17.20 (IO19)
- net PD3 renamed VD27
- net VD27: now also U23.5 (A3)
- net PD30 renamed VD6
- net VD6: no longer U17.19 (IO20)
- net PD31 renamed VD7
- net VD7: no longer U17.18 (IO21)
- net PD4 renamed VD28
- net VD28: now also U23.6 (A4)
- net PD5 renamed VD29
- net VD29: now also U23.7 (A5)
- net PD6 renamed VD30
- net VD30: now also U23.8 (A6)
- net PD7 renamed VD31
- net VD31: now also U23.9 (A7)
- net PD8 renamed VD16
- net VD16: now also U22.2 (A0)
- net PD9 renamed VD17
- net VD17: now also U22.3 (A1)
- net ~{PDBEN} renamed ~{PB32}
- net ~{PB32}: now also U17.11 (IO3); no longer U4.19 (CE)
- net ~{SDReady}: no longer names the net of U13.4
- net ~{SDReady}: no longer U17.12 (IO1)
- net ~{SysClk-5v}: no longer names the net of U9.12
- net ~{SysClk-5v}: no longer U11.194 (SCLK)
- new net VID-M/~{IO}: U11.8 (SM/~{IO}), U17.21 (IO17)
- new net ~{PBE0}: U17.5 (IO14), U4.19 (CE)
- new net ~{PBE1}: U17.6 (IO11), U8.19 (CE)
- new net ~{PBE2}: U17.9 (IO4), U22.19 (CE)
- new net ~{PBE3}: U17.8 (IO5), U23.19 (CE)
- no-connect marks 2 -> 0
Other:
- note added: "CPU"
- note added: "Clock & Reset"
- note added: "Expansion Bus"
- note added: "PS/2 Keyboard/Mouse"
- note added: "Peripheral Bus Control"
- note added: "Power"
- note added: "ROM/RAM"
- note added: "Serial"
- note added: "Video"
- note removed: "ADS-Q0"
- note removed: "ADS-Q1"
- moved on the sheet: C13, C14, C15, C16, C17, C18, C19, C20, C21, C22, C23, C24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

Commit message: New peripheral bus debugging
- add pull-ups to bus transceiver enable signals for debugging
- change reset pull-up to 1k to help with rise times
- update bank registers configuration for new peripheral bus
Parts:
- added RN7: 9A103J, Resistor_THT:R_Array_SIP9, symbol Device:R_Network08_US
- RN3: value 10X-1-472LF -> 10X-1-102LF
Connections:
- net +5V: now also RN7.1 (common)
- net ~{PB32}: now also RN7.2 (R1)
- net ~{PBE0}: now also RN7.6 (R5)
- net ~{PBE1}: now also RN7.5 (R4)
- net ~{PBE2}: now also RN7.3 (R2)
- net ~{PBE3}: now also RN7.4 (R3)
Changed lines of the file:
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@@
 	(wire
 		(pts
+			(xy 152.4 416.56) (xy 165.1 416.56)
+		)
+		(stroke
+			(width 0)
+			(type default)
+		)
+	)
+	(wire
+		(pts
 			(xy 645.16 246.38) (xy 657.86 246.38)
 		)
@@
 	(wire
 		(pts
+			(xy 152.4 414.02) (xy 165.1 414.02)
+		)
+		(stroke
+			(width 0)
+			(type default)
+		)
+	)
+	(wire
+		(pts
 			(xy 241.3 309.88) (xy 254 309.88)
 		)
@@
 	(wire
 		(pts
+			(xy 152.4 408.94) (xy 165.1 408.94)
+		)
+		(stroke
+			(width 0)
+			(type default)
+		)
+	)
+	(wire
+		(pts
 			(xy 368.3 314.96) (xy 381 314.96)
 		)
@@
 	(wire
 		(pts
+			(xy 152.4 419.1) (xy 165.1 419.1)
+		)
+		(stroke
+			(width 0)
+			(type default)
+		)
+	)
+	(wire
+		(pts
 			(xy 622.3 406.4) (xy 609.6 406.4)
 		)
@@
 	(wire
 		(pts
+			(xy 152.4 411.48) (xy 165.1 411.48)
+		)
+		(stroke
+			(width 0)
+			(type default)
+		)
+	)
+	(wire
+		(pts
 			(xy 520.7 327.66) (xy 533.4 327.66)
 		)
@@
 		)
 	)
+	(label "~{PBE3}"
+		(at 152.4 414.02 0)
+		(effects
+			(font
+				(size 1.27 1.27)
+			)
+			(justify left bottom)
+		)
+	)
 	(label "A25"
 		(at 142.24 91.44 180)
@@
 		)
 	)
+	(label "~{PBE1}"
+		(at 152.4 416.56 0)
+		(effects
+			(font
+				(size 1.27 1.27)
+			)
+			(justify left bottom)
+		)
+	)
 	(label "VD9"
 		(at 505.46 203.2 180)
@@
 		)
 	)
+	(label "~{PBE2}"
+		(at 152.4 411.48 0)
+		(effects
+			(font
+				(size 1.27 1.27)
+			)
+			(justify left bottom)
+		)
+	)
 	(label "D22"
 		(at 78.74 83.82 180)
@@
 		)
 	)
+	(label "~{PB32}"
+		(at 152.4 408.94 0)
+		(effects
+			(font
+				(size 1.27 1.27)
+			)
+			(justify left bottom)
+		)
+	)
 	(label "VD22"
 		(at 203.2 373.38 0)
@@
 		)
 	)
+	(label "~{PBE0}"
+		(at 152.4 419.1 0)
+		(effects
+			(font
+				(size 1.27 1.27)
+			)
+			(justify left bottom)
+		)
+	)
 	(label "VMD39"
 		(at 607.06 408.94 180)
@@
 	)
 	(symbol
+		(lib_id "Device:R_Network08_US")
+		(at 170.18 419.1 270)
+		(unit 1)
+		(exclude_from_sim no)
+		(in_bom yes)
+		(on_board yes)
+		(dnp no)
+		(fields_autoplaced yes)
+		(property "Reference" "RN7"
+			(at 169.926 403.5255 90)
+			(effects
+				(font
+					(size 1.27 1.27)
+				)
+			)
+		)
+		(property "Value" "9A103J"
+			(at 169.926 405.9498 90)
+			(effects
+				(font
+					(size 1.27 1.27)
+				)
+			)
+		)
+		(property "Footprint" "Resistor_THT:R_Array_SIP9"
+			(at 170.18 431.165 90)
+			(effects
+				(font
+					(size 1.27 1.27)
+				)
+				(hide yes)
+			)
+		)
+		(property "Datasheet" "http://www.vishay.com/docs/31509/csc.pdf"
+			(at 170.18 419.1 0)
+			(effects
+				(font
+					(size 1.27 1.27)
+				)
+				(hide yes)
+			)
+		)
+		(property "Description" "8 resistor network, star topology, bussed resistors, small US symbol"
+			(at 170.18 419.1 0)
+			(effects
+				(font
+					(size 1.27 1.27)
+				)
+				(hide yes)
+			)
+		)
+		(pin "5"
+		)
+		(pin "8"
+		)
+		(pin "7"
+		)
+		(pin "3"
+		)
+		(pin "1"
+		)
+		(pin "4"
+		)
+		(pin "6"
+		)
+		(pin "2"
+		)
+		(pin "9"
+		)
+		(instances
+			(project "PikaPC_Mainboard"
+				(path "/31647a00-1631-4687-a4ca-8a073377aae5"
+					(reference "RN7")
+					(unit 1)
+				)
+			)
+		)
+	)
+	(symbol
 		(lib_id "Oscillator:CXO_DIP8")
 		(at 190.5 259.08 0)
@@
 	)
 	(symbol
+		(lib_id "power:+5V")
+		(at 175.26 408.94 270)
+		(unit 1)
+		(exclude_from_sim no)
+		(in_bom yes)
+		(on_board yes)
+		(dnp no)
+		(fields_autoplaced yes)
+		(property "Reference" "#PWR029"
+			(at 171.45 408.94 0)
+			(effects
+				(font
+					(size 1.27 1.27)
+				)
+				(hide yes)
+			)
+		)
+		(property "Value" "+5V"
+			(at 178.435 408.94 90)
+			(effects
+				(font
+					(size 1.27 1.27)
+				)
+				(justify left)
+			)
+		)
+		(property "Footprint" ""
+			(at 175.26 408.94 0)
+			(effects
+				(font
+					(size 1.27 1.27)
+				)
+				(hide yes)
+			)
+		)
+		(property "Datasheet" ""
+			(at 175.26 408.94 0)
+			(effects
+				(font
+					(size 1.27 1.27)
+				)
+				(hide yes)
+			)
+		)
+		(property "Description" "Power symbol creates a global label with name \"+5V\""
+			(at 175.26 408.94 0)
+			(effects
+				(font
+					(size 1.27 1.27)
+				)
+				(hide yes)
+			)
+		)
+		(pin "1"
+		)
+		(instances
+			(project "PikaPC_Mainboard"
+				(path "/31647a00-1631-4687-a4ca-8a073377aae5"
+					(reference "#PWR029")
+					(unit 1)
+				)
+			)
+		)
+	)
+	(symbol
 		(lib_id "74xx:74LVC125")
 		(at 320.04 416.56 0)
@@
 			)
 		)
-		(property "Value" "10X-1-472LF"
+		(property "Value" "10X-1-102LF"
 			(at 246.126 75.7498 90)
 			(effects

Commit message: VRAM control debugging
- add strapping resistors for slow vram cycles
- fix swapped CAS2 & CAS3 pins on ViRGE symbol
Parts:
- added RN8: 9A103J, Resistor_THT:R_Array_SIP9, symbol Device:R_Network08_US
- RN7: value 9A103J -> 10X-1-472F
Connections:
- net GND: now also RN8.1 (common)
- net VMD16: now also RN8.2 (R1)
- net VMD17: now also RN8.3 (R2)
- net VMD18: now also RN8.4 (R3)
- net VMD19: now also RN8.5 (R4)
- net ~{VMCAS2}: now also U11.83 (~{CAS2}); no longer U11.82 (~{CAS3})
- net ~{VMCAS3}: now also U11.82 (~{CAS3}); no longer U11.83 (~{CAS2})
Other:
- note added: "RN8 for slow VRAM cycles"
- moved on the sheet: RN6
