File: Hardware/PikaPC_SIMM72/PikaPC_SIMM72.kicad_pcb (KiCad board)
At the start: 2 copper layers, 101.6 x 101.6 mm, 364 parts, among them J1 DIN41612_03x32_C_Split, J2 TE-822021-4, J3 Conn_02x07_Odd_Even, U1 74F521, U2 ATF1508AS, U3 74FCT2245, U4 74FCT2245, U5 74FCT2245, U6 74FCT2245

Commit message: Un-assign main bus pins 22 & 23
Parts:
- R10, R11, R12, R13, R14, R15, R16, R17, R18, R19, R20, R21, R22, R23, R24, R25, R8, R9: value 4k7 -> 33R
Connections:
- J1 pad b22: GND -> unconnected-(J1B-Pin_b22-Padb22)
- J1 pad b23: GND -> unconnected-(J1B-Pin_b23-Padb23)

Commit message: Prep for output
Other:
- board text added: "72-PIN SIMM"
