File: Hardware/PikaPC_ViRGE/Video.kicad_sch (KiCad schematic)
At the start: 16 parts, among them J3 Conn_02x08_Odd_Even, J4 DE15_Socket_HighDensity_Mount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, U2 86C325, Y1 14M31818

Commit message: ViRGE card PCB layout
Parts:
- renumbered U2 to U1
Changed lines of the file:
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@@
 		(dnp no)
 		(fields_autoplaced yes)
-		(property "Reference" "U2"
+		(property "Reference" "U1"
 			(at 203.2 24.13 0)
 			(do_not_autoplace yes)
@@
 			(project "PikaPC_ViRGE"
 				(path "/dd18a86c-f3c8-46f4-a73e-5b02d2ebb148/b46edc01-5753-425d-92b9-4f18e9204e38"
-					(reference "U2")
+					(reference "U1")
 					(unit 4)
 				)
@@
 		(dnp no)
 		(fields_autoplaced yes)
-		(property "Reference" "U2"
+		(property "Reference" "U1"
 			(at 50.8 36.83 0)
 			(do_not_autoplace yes)
@@
 			(project "PikaPC_ViRGE"
 				(path "/dd18a86c-f3c8-46f4-a73e-5b02d2ebb148/b46edc01-5753-425d-92b9-4f18e9204e38"
-					(reference "U2")
+					(reference "U1")
 					(unit 3)
 				)

Commit message: Prep for output
Parts:
- C2: Mouser (none) -> 187-CL21B104KACNNNC
- FB1, FB2, FB3: footprint Inductor_THT:L_Axial_L7.0mm_D3.3mm_P5.08mm_Vertical_Fastron_MICC -> Inductor_THT:L_Axial_L5.3mm_D2.2mm_P2.54mm_Vertical_Vishay_IM-1; symbol Device:FerriteBead -> Device:FerriteBead_Small
- J3: now not fitted
- J4: footprint Connector_Dsub:DSUB-15-HD_Socket_Horizontal_P2.29x1.90mm_EdgePinOffset3.03mm_Housed_MountingHolesOffset4.94mm -> PikaPC_ViRGE:DE15 (EDAC 634-015); Mouser (none) -> 587-634-015-263-032
- R10, R8, R9: Mouser (none) -> 603-RC0805FR-1375RL
- R11, R12, R13, R14, R15: Mouser (none) -> 303-0805S8J0103T5E
Other:
- moved on the sheet: FB1, FB2, FB3
Changed lines of the file:
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@@
 	(wire
 		(pts
-			(xy 53.34 68.58) (xy 71.12 68.58)
+			(xy 53.34 68.58) (xy 66.04 68.58)
 		)
 		(stroke
@@
 	(wire
 		(pts
-			(xy 53.34 58.42) (xy 71.12 58.42)
+			(xy 53.34 58.42) (xy 66.04 58.42)
 		)
 		(stroke
@@
 	(wire
 		(pts
-			(xy 33.02 63.5) (xy 45.72 63.5)
+			(xy 35.56 63.5) (xy 48.26 63.5)
 		)
 		(stroke
@@
 	(wire
 		(pts
-			(xy 53.34 63.5) (xy 71.12 63.5)
+			(xy 53.34 63.5) (xy 66.04 63.5)
 		)
 		(stroke
@@
 	(wire
 		(pts
-			(xy 33.02 68.58) (xy 45.72 68.58)
+			(xy 35.56 68.58) (xy 48.26 68.58)
 		)
 		(stroke
@@
 	(wire
 		(pts
-			(xy 33.02 58.42) (xy 45.72 58.42)
+			(xy 35.56 58.42) (xy 48.26 58.42)
 		)
 		(stroke
@@
 	)
 	(label "Vid-G-Out"
-		(at 71.12 63.5 180)
+		(at 66.04 63.5 180)
 		(effects
 			(font
@@
 	)
 	(label "Vid-G"
-		(at 33.02 63.5 0)
+		(at 35.56 63.5 0)
 		(effects
 			(font
@@
 	)
 	(label "Vid-B"
-		(at 33.02 68.58 0)
+		(at 35.56 68.58 0)
 		(effects
 			(font
@@
 	)
 	(label "Vid-R"
-		(at 33.02 58.42 0)
+		(at 35.56 58.42 0)
 		(effects
 			(font
@@
 	)
 	(label "Vid-B-Out"
-		(at 71.12 68.58 180)
+		(at 66.04 68.58 180)
 		(effects
 			(font
@@
 	)
 	(label "Vid-R-Out"
-		(at 71.12 58.42 180)
+		(at 66.04 58.42 180)
 		(effects
 			(font
@@
 			)
 		)
+		(property "Mouser" "303-0805S8J0103T5E "
+			(at 218.44 106.68 90)
+			(effects
+				(font
+					(size 1.27 1.27)
+				)
+				(hide yes)
+			)
+		)
 		(pin "1"
 		)
@@
 	)
 	(symbol
-		(lib_id "Device:FerriteBead")
-		(at 49.53 58.42 270)
+		(lib_id "Device:FerriteBead_Small")
+		(at 50.8 58.42 270)
 		(unit 1)
 		(exclude_from_sim no)
@@
 		(dnp no)
 		(property "Reference" "FB1"
-			(at 46.99 57.15 90)
+			(at 48.26 57.15 90)
 			(effects
 				(font
@@
 		)
 		(property "Value" "FerriteBead"
-			(at 55.88 59.69 90)
+			(at 57.15 59.69 90)
 			(effects
 				(font
@@
 			)
 		)
-		(property "Footprint" "Inductor_THT:L_Axial_L7.0mm_D3.3mm_P5.08mm_Vertical_Fastron_MICC"
-			(at 49.53 56.642 90)
+		(property "Footprint" "Inductor_THT:L_Axial_L5.3mm_D2.2mm_P2.54mm_Vertical_Vishay_IM-1"
+			(at 50.8 56.642 90)
 			(effects
 				(font
@@
 		)
 		(property "Datasheet" "~"
-			(at 49.53 58.42 0)
+			(at 50.8 58.42 0)
 			(effects
 				(font
@@
 			)
 		)
-		(property "Description" "Ferrite bead"
-			(at 49.53 58.42 0)
+		(property "Description" "Ferrite bead, small symbol"
+			(at 50.8 58.42 0)
 			(effects
 				(font
@@
 			)
 		)
+		(property "Mouser" "187-CL21B104KACNNNC"
+			(at 147.32 76.2 90)
+			(effects
+				(font
+					(size 1.27 1.27)
+				)
+				(hide yes)
+			)
+		)
 		(pin "2"
 		)
@@
 			)
 		)
+		(property "Mouser" "303-0805S8J0103T5E "
+			(at 218.44 109.22 90)
+			(effects
+				(font
+					(size 1.27 1.27)
+				)
+				(hide yes)
+			)
+		)
 		(pin "1"
 		)
@@
 	)
 	(symbol
-		(lib_id "Device:FerriteBead")
-		(at 49.53 63.5 270)
+		(lib_id "Device:FerriteBead_Small")
+		(at 50.8 63.5 270)
 		(unit 1)
 		(exclude_from_sim no)
@@
 		(dnp no)
 		(property "Reference" "FB2"
-			(at 46.99 62.23 90)
+			(at 48.26 62.23 90)
 			(effects
 				(font
@@
 		)
 		(property "Value" "FerriteBead"
-			(at 55.88 64.77 90)
+			(at 57.15 64.77 90)
 			(effects
 				(font
@@
 			)
 		)
-		(property "Footprint" "Inductor_THT:L_Axial_L7.0mm_D3.3mm_P5.08mm_Vertical_Fastron_MICC"
-			(at 49.53 61.722 90)
+		(property "Footprint" "Inductor_THT:L_Axial_L5.3mm_D2.2mm_P2.54mm_Vertical_Vishay_IM-1"
+			(at 50.8 61.722 90)
 			(effects
 				(font
@@
 		)
 		(property "Datasheet" "~"
-			(at 49.53 63.5 0)
+			(at 50.8 63.5 0)
 			(effects
 				(font
@@
 			)
 		)
-		(property "Description" "Ferrite bead"
-			(at 49.53 63.5 0)
+		(property "Description" "Ferrite bead, small symbol"
+			(at 50.8 63.5 0)
 			(effects
 				(font
@@
 			)
 		)
+		(property "Mouser" "303-0805S8J0103T5E "
+			(at 218.44 99.06 90)
+			(effects
+				(font
+					(size 1.27 1.27)
+				)
+				(hide yes)
+			)
+		)
 		(pin "1"
 		)
@@
 			)
 		)
+		(property "Mouser" "603-RC0805FR-1375RL"
+			(at 85.09 58.42 90)
+			(effects
+				(font
+					(size 1.27 1.27)
+				)
+				(hide yes)
+			)
+		)
 		(pin "1"
 		)
@@
 			)
 		)
+		(property "Mouser" "303-0805S8J0103T5E "
+			(at 218.44 104.14 90)
+			(effects
+				(font
+					(size 1.27 1.27)
+				)
+				(hide yes)
+			)
+		)
 		(pin "1"
 		)
@@
 			)
 		)
+		(property "Mouser" "603-RC0805FR-1375RL"
+			(at 82.55 58.42 90)
+			(effects
+				(font
+					(size 1.27 1.27)
+				)
+				(hide yes)
+			)
+		)
 		(pin "1"
 		)
@@
 	)
 	(symbol
-		(lib_id "Device:FerriteBead")
-		(at 49.53 68.58 270)
+		(lib_id "Device:FerriteBead_Small")
+		(at 50.8 68.58 270)
 		(unit 1)
 		(exclude_from_sim no)
@@
 		(dnp no)
 		(property "Reference" "FB3"
-			(at 46.99 67.31 90)
+			(at 48.26 67.31 90)
 			(effects
 				(font
@@
 		)
 		(property "Value" "FerriteBead"
-			(at 55.88 69.85 90)
+			(at 57.15 69.85 90)
 			(effects
 				(font
@@
 			)
 		)
-		(property "Footprint" "Inductor_THT:L_Axial_L7.0mm_D3.3mm_P5.08mm_Vertical_Fastron_MICC"
-			(at 49.53 66.802 90)
+		(property "Footprint" "Inductor_THT:L_Axial_L5.3mm_D2.2mm_P2.54mm_Vertical_Vishay_IM-1"
+			(at 50.8 66.802 90)
 			(effects
 				(font
@@
 		)
 		(property "Datasheet" "~"
-			(at 49.53 68.58 0)
+			(at 50.8 68.58 0)
 			(effects
 				(font
@@
 			)
 		)
-		(property "Description" "Ferrite bead"
-			(at 49.53 68.58 0)
+		(property "Description" "Ferrite bead, small symbol"
+			(at 50.8 68.58 0)
 			(effects
 				(font
@@
 			)
 		)
-		(property "Footprint" "Connector_Dsub:DSUB-15-HD_Socket_Horizontal_P2.29x1.90mm_EdgePinOffset3.03mm_Housed_MountingHolesOffset4.94mm"
+		(property "Footprint" "PikaPC_ViRGE:DE15 (EDAC 634-015)"
 			(at 34.29 114.3 0)
 			(effects
@@
 			)
 		)
+		(property "Mouser" "587-634-015-263-032 "
+			(at 58.42 124.46 0)
+			(effects
+				(font
+					(size 1.27 1.27)
+				)
+				(hide yes)
+			)
+		)
 		(pin "8"
 		)
@@
 		(in_bom yes)
 		(on_board yes)
-		(dnp no)
+		(dnp yes)
 		(fields_autoplaced yes)
 		(property "Reference" "J3"
@@
 			)
 		)
+		(property "Mouser" "603-RC0805FR-1375RL"
+			(at 87.63 58.42 90)
+			(effects
+				(font
+					(size 1.27 1.27)
+				)
+				(hide yes)
+			)
+		)
 		(pin "1"
 		)
@@
 			(effects
 				(font
+					(size 1.27 1.27)
+				)
+				(hide yes)
+			)
+		)
+		(property "Mouser" "303-0805S8J0103T5E "
+			(at 218.44 101.6 90)
+			(effects
+				(font
