File: Hardware/PikaPC_ViRGE/power.kicad_sch (KiCad schematic)
At the start: 27 parts, among them U1 ATF1504, U2 86C325

Commit message: ViRGE card PCB layout
Parts:
- U2: renamed from U1; value ATF1504 -> ATF1504AS
- renumbered U2 to U1
Changed lines of the file:
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@@
 		(dnp no)
 		(fields_autoplaced yes)
-		(property "Reference" "U1"
+		(property "Reference" "U2"
 			(at 182.88 24.13 0)
 			(do_not_autoplace yes)
@@
 			)
 		)
-		(property "Value" "ATF1504"
+		(property "Value" "ATF1504AS"
 			(at 198.12 24.13 0)
 			(do_not_autoplace yes)
@@
 			(project "PikaPC_ViRGE"
 				(path "/dd18a86c-f3c8-46f4-a73e-5b02d2ebb148/9b83794d-ac83-444e-b108-8beac34e7e90"
-					(reference "U1")
+					(reference "U2")
 					(unit 2)
 				)
@@
 		(dnp no)
 		(fields_autoplaced yes)
-		(property "Reference" "U2"
+		(property "Reference" "U1"
 			(at 63.5 24.13 0)
 			(do_not_autoplace yes)
@@
 			(project "PikaPC_ViRGE"
 				(path "/dd18a86c-f3c8-46f4-a73e-5b02d2ebb148/9b83794d-ac83-444e-b108-8beac34e7e90"
-					(reference "U2")
+					(reference "U1")
 					(unit 5)
 				)

Commit message: Prep for output
Parts:
- added R38: 147R, Resistor_SMD:R_0805_2012Metric, symbol Device:R_Small_US
- C10, C11, C12, C13, C14, C15, C19, C20, C21, C3, C4, C48, C5, C6, C7, C8, C9: Mouser (none) -> 187-CL21B104KACNNNC
- C16, C17, C22: Mouser (none) -> 187-CL21B105KOFNNNG
- L1, L2: Mouser (none) -> 708-RMCF1210ZT0R00
- R16, R17: now not fitted
Connections:
- net GNDA: now also R38.1
- net RSET: now also R38.2
Other:
- note added: "R38 is ideal value for RSET R16 & R17 are alternates that approximate 147Ω"
- note removed: "RSET Target: 147R"
