File: Hardware/PikaPC_ViRGE/main_bus.kicad_sch (KiCad schematic)
At the start: 13 parts, among them J1 Conn_02x07_Odd_Even, J2 DIN41612_03x32_C_Split, U1 ATF1504, U2 86C325, U3 74F521

Commit message: ViRGE card PCB layout
Parts:
- added IO11, IO16, IO2, IO24, IO30, IO44, IO5: TestPoint, Connector_PinHeader_2.54mm:PinHeader_1x01_P2.54mm_Vertical, symbol Connector:TestPoint
- U2: renamed from U1; value ATF1504 -> ATF1504AS
- renumbered J2 to J1, J1 to J2, U2 to U1
Connections:
- net A23: now also U2.18 (IO21); no longer U2.26 (IO36)
- net A24: now also U2.19 (IO20); no longer U2.27 (IO37)
- net Bus-R/~{W}: now also U2.36 (IO52); no longer U2.20 (IO19)
- net INT0: now also U2.9 (IO4); no longer U2.37 (IO53)
- net VID-M/~{IO}: now also U2.37 (IO53); no longer U2.29 (IO41)
- net VID-SAUP1: now also U2.5 (IO14); no longer U2.24 (IO33)
- net VID-SAUP2: now also U2.11 (IO3); no longer U2.25 (IO35)
- net ~{AEN}: now also U2.33 (IO49); no longer U2.14 (IO30)
- net ~{BEN}: now also U2.25 (IO35); no longer U2.17 (IO24)
- net ~{Bus-ACK}: now also U2.20 (IO19); no longer U2.19 (IO20)
- net ~{Bus-BRACK}: now also U2.26 (IO36); no longer U2.5 (IO14)
- net ~{Bus-BURST}: now also U2.24 (IO33); no longer U2.6 (IO11)
- net ~{Bus-IACK}: now also U2.34 (IO51); no longer U2.8 (IO5)
- net ~{Bus-IRQ0}: now also U2.31 (IO46); no longer U2.12 (IO1)
- net ~{Bus-IRQ1}: now also U2.29 (IO41); no longer U2.11 (IO3)
- net ~{Bus-IRQ2}: now also U2.27 (IO37); no longer U2.9 (IO4)
- net ~{Bus-Start}: now also U2.21 (IO17); no longer U2.18 (IO21)
- net ~{OE}: now also U2.12 (IO1); no longer U2.31 (IO46)
- net ~{VID-ADS}: now also U2.41 (IO64); no longer U2.33 (IO49)
- net ~{VID-RDYIN}: now also U2.39 (IO57); no longer U2.34 (IO51)
- net ~{VID-SRDY}: now also U2.40 (IO62); no longer U2.36 (IO52)
- net at U2.2 (OE2/GCLK2): now also IO2.1
- net at U2.4 (IO16): now also IO16.1
- net at U2.44 (OE1): now also IO44.1
- new net: IO24.1, U2.17 (IO24)
- new net: IO11.1, U2.6 (IO11)
- new net: IO30.1, U2.14 (IO30)
- new net: IO5.1, U2.8 (IO5)

Commit message: Un-assign main bus pins 22 & 23
Connections:
- net GND: no longer J1.b22 (Pin_b22), J1.b23 (Pin_b23)
Changed lines of the file:
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@@
 	)
 	(symbol
-		(lib_id "power:GND")
-		(at 208.28 81.28 270)
-		(unit 1)
-		(exclude_from_sim no)
-		(in_bom yes)
-		(on_board yes)
-		(dnp no)
-		(fields_autoplaced yes)
-		(property "Reference" "#PWR035"
-			(at 201.93 81.28 0)
-			(effects
-				(font
-					(size 1.27 1.27)
-				)
-				(hide yes)
-			)
-		)
-		(property "Value" "GND"
-			(at 205.1051 81.28 90)
-			(effects
-				(font
-					(size 1.27 1.27)
-				)
-				(justify right)
-			)
-		)
-		(property "Footprint" ""
-			(at 208.28 81.28 0)
-			(effects
-				(font
-					(size 1.27 1.27)
-				)
-				(hide yes)
-			)
-		)
-		(property "Datasheet" ""
-			(at 208.28 81.28 0)
-			(effects
-				(font
-					(size 1.27 1.27)
-				)
-				(hide yes)
-			)
-		)
-		(property "Description" "Power symbol creates a global label with name \"GND\" , ground"
-			(at 208.28 81.28 0)
-			(effects
-				(font
-					(size 1.27 1.27)
-				)
-				(hide yes)
-			)
-		)
-		(pin "1"
-		)
-		(instances
-			(project "PikaPC_ViRGE"
-				(path "/dd18a86c-f3c8-46f4-a73e-5b02d2ebb148/b87e7203-ea3a-46a7-9e06-4b89d81b9033"
-					(reference "#PWR035")
-					(unit 1)
-				)
-			)
-		)
-	)
-	(symbol
 		(lib_id "PikaPC:S3 86C325 ViRGE")
 		(at 119.38 22.86 0)
@@
 					(unit 1)
 				)
-			)
-		)
-	)
-	(symbol
-		(lib_id "power:GND")
-		(at 208.28 83.82 270)
-		(unit 1)
-		(exclude_from_sim no)
-		(in_bom yes)
-		(on_board yes)
-		(dnp no)
-		(fields_autoplaced yes)
-		(property "Reference" "#PWR036"
-			(at 201.93 83.82 0)
-			(effects
-				(font
-					(size 1.27 1.27)
-				)
-				(hide yes)
-			)
-		)
-		(property "Value" "GND"
-			(at 205.1051 83.82 90)
-			(effects
-				(font
-					(size 1.27 1.27)
-				)
-				(justify right)
-			)
-		)
-		(property "Footprint" ""
-			(at 208.28 83.82 0)
-			(effects
-				(font
-					(size 1.27 1.27)
-				)
-				(hide yes)
-			)
-		)
-		(property "Datasheet" ""
-			(at 208.28 83.82 0)
-			(effects
-				(font
-					(size 1.27 1.27)
-				)
-				(hide yes)
-			)
-		)
-		(property "Description" "Power symbol creates a global label with name \"GND\" , ground"
-			(at 208.28 83.82 0)
-			(effects
-				(font
-					(size 1.27 1.27)
-				)
-				(hide yes)
-			)
-		)
-		(pin "1"
-		)
-		(instances
-			(project "PikaPC_ViRGE"
-				(path "/dd18a86c-f3c8-46f4-a73e-5b02d2ebb148/b87e7203-ea3a-46a7-9e06-4b89d81b9033"
-					(reference "#PWR036")
-					(unit 1)
-				)

Commit message: Prep for output
Parts:
- C1: Mouser (none) -> 187-CL21B104KACNNNC
- R1, R2, R3, R4, R5, R6, R7: Mouser (none) -> 303-0805W8J0472T5E
Changed lines of the file:
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@@
 			)
 		)
+		(property "Mouser" "303-0805W8J0472T5E"
+			(at 88.9 175.26 90)
+			(effects
+				(font
+					(size 1.27 1.27)
+				)
+				(hide yes)
+			)
+		)
 		(pin "1"
 		)
@@
 			)
 		)
+		(property "Mouser" "303-0805W8J0472T5E"
+			(at 88.9 170.18 90)
+			(effects
+				(font
+					(size 1.27 1.27)
+				)
+				(hide yes)
+			)
+		)
 		(pin "1"
 		)
@@
 			)
 		)
+		(property "Mouser" "303-0805W8J0472T5E"
+			(at 88.9 180.34 90)
+			(effects
+				(font
+					(size 1.27 1.27)
+				)
+				(hide yes)
+			)
+		)
 		(pin "1"
 		)
@@
 			)
 		)
+		(property "Mouser" "303-0805W8J0472T5E"
+			(at 88.9 172.72 90)
+			(effects
+				(font
+					(size 1.27 1.27)
+				)
+				(hide yes)
+			)
+		)
 		(pin "1"
 		)
@@
 			)
 		)
+		(property "Mouser" "187-CL21B104KACNNNC"
+			(at 132.08 153.67 90)
+			(effects
+				(font
+					(size 1.27 1.27)
+				)
+				(hide yes)
+			)
+		)
 		(pin "2"
 		)
@@
 			)
 		)
+		(property "Mouser" "303-0805W8J0472T5E"
+			(at 88.9 165.1 90)
+			(effects
+				(font
+					(size 1.27 1.27)
+				)
+				(hide yes)
+			)
+		)
 		(pin "1"
 		)
@@
 			)
 		)
+		(property "Mouser" "303-0805W8J0472T5E"
+			(at 88.9 167.64 90)
+			(effects
+				(font
+					(size 1.27 1.27)
+				)
+				(hide yes)
+			)
+		)
 		(pin "1"
 		)
@@
 			(effects
 				(font
+					(size 1.27 1.27)
+				)
+				(hide yes)
+			)
+		)
+		(property "Mouser" "303-0805W8J0472T5E"
+			(at 88.9 177.8 90)
+			(effects
+				(font

Commit message: add missing pull-ups on SRDY# & RDYIN#
Parts:
- added R39, R40: 10K, Resistor_SMD:R_0805_2012Metric, symbol Device:R_Small_US
Connections:
- net +5V: now also R39.1, R40.1
- net ~{VID-RDYIN}: now also R39.2
- net ~{VID-SRDY}: now also R40.2

Commit message: Add pull-up to LOCA# on ViRGE card
Parts:
- added R41: 10K, Resistor_SMD:R_0805_2012Metric, symbol Device:R_Small_US
Connections:
- net +5V: now also R41.2
- net ~{VID-LOCA}: now also R41.1
Changed lines of the file:
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@@
 	(wire
 		(pts
+			(xy 160.02 109.22) (xy 160.02 106.68)
+		)
+		(stroke
+			(width 0)
+			(type default)
+		)
+	)
+	(wire
+		(pts
 			(xy 38.1 144.78) (xy 50.8 144.78)
 		)
@@
 	(wire
 		(pts
-			(xy 137.16 109.22) (xy 149.86 109.22)
+			(xy 137.16 109.22) (xy 152.4 109.22)
 		)
 		(stroke
@@
 	(wire
 		(pts
+			(xy 157.48 109.22) (xy 160.02 109.22)
+		)
+		(stroke
+			(width 0)
+			(type default)
+		)
+	)
+	(wire
+		(pts
 			(xy 38.1 101.6) (xy 50.8 101.6)
 		)
@@
 	)
 	(symbol
+		(lib_id "Device:R_Small_US")
+		(at 154.94 109.22 90)
+		(unit 1)
+		(exclude_from_sim no)
+		(in_bom yes)
+		(on_board yes)
+		(dnp no)
+		(property "Reference" "R41"
+			(at 151.13 107.95 90)
+			(effects
+				(font
+					(size 1.27 1.27)
+				)
+			)
+		)
+		(property "Value" "10K"
+			(at 158.75 107.95 90)
+			(effects
+				(font
+					(size 1.27 1.27)
+				)
+			)
+		)
+		(property "Footprint" "Resistor_SMD:R_0805_2012Metric"
+			(at 154.94 109.22 0)
+			(effects
+				(font
+					(size 1.27 1.27)
+				)
+				(hide yes)
+			)
+		)
+		(property "Datasheet" ""
+			(at 154.94 109.22 0)
+			(effects
+				(font
+					(size 1.27 1.27)
+				)
+				(hide yes)
+			)
+		)
+		(property "Description" ""
+			(at 154.94 109.22 0)
+			(effects
+				(font
+					(size 1.27 1.27)
+				)
+				(hide yes)
+			)
+		)
+		(property "Mouser" "303-0805S8J0103T5E "
+			(at 154.94 109.22 90)
+			(effects
+				(font
+					(size 1.27 1.27)
+				)
+				(hide yes)
+			)
+		)
+		(pin "1"
+		)
+		(pin "2"
+		)
+		(instances
+			(project "PikaPC_ViRGE"
+				(path "/dd18a86c-f3c8-46f4-a73e-5b02d2ebb148/b87e7203-ea3a-46a7-9e06-4b89d81b9033"
+					(reference "R41")
+					(unit 1)
+				)
+			)
+		)
+	)
+	(symbol
 		(lib_id "power:GND")
 		(at 241.3 27.94 270)
@@
 					(unit 1)
 				)
+			)
+		)
+	)
+	(symbol
+		(lib_id "power:+5V")
+		(at 160.02 106.68 0)
+		(unit 1)
+		(exclude_from_sim no)
+		(in_bom yes)
+		(on_board yes)
+		(dnp no)
+		(fields_autoplaced yes)
+		(property "Reference" "#PWR0147"
+			(at 160.02 110.49 0)
+			(effects
+				(font
+					(size 1.27 1.27)
+				)
+				(hide yes)
+			)
+		)
+		(property "Value" "+5V"
+			(at 160.02 102.5469 0)
+			(effects
+				(font
+					(size 1.27 1.27)
+				)
+			)
+		)
+		(property "Footprint" ""
+			(at 160.02 106.68 0)
+			(effects
+				(font
+					(size 1.27 1.27)
+				)
+				(hide yes)
+			)
+		)
+		(property "Datasheet" ""
+			(at 160.02 106.68 0)
+			(effects
+				(font
+					(size 1.27 1.27)
+				)
+				(hide yes)
+			)
+		)
+		(property "Description" "Power symbol creates a global label with name \"+5V\""
+			(at 160.02 106.68 0)
+			(effects
+				(font
+					(size 1.27 1.27)
+				)
+				(hide yes)
+			)
+		)
+		(pin "1"
+		)
+		(instances
+			(project "PikaPC_ViRGE"
+				(path "/dd18a86c-f3c8-46f4-a73e-5b02d2ebb148/b87e7203-ea3a-46a7-9e06-4b89d81b9033"
+					(reference "#PWR0147")
+					(unit 1)
+				)
