File: Hardware/PikaPC_IDE/PikaPC_IDE.kicad_pcb (KiCad board)
At the start: 2 copper layers, 101.6 x 101.6 mm, 208 parts, among them J1 DIN41612_03x32_C_Split, J2 Conn_02x08_Odd_Even, J3 Conn_02x03_Odd_Even, J4 Conn_02x03_Odd_Even, J5 Conn_01x06, J6 Conn_01x04, U1 74FCT2245, U2 74FCT2245, U3 74AHCT573, U4 74LS139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

Commit message: Add prototyping card
Routing:
- net unconnected-(IDE1-Pin_21-Pad21): track 13.8 -> 0.00 mm
- net unconnected-(IDE1-Pin_34-Pad34): track 13.8 -> 0.00 mm
- net unconnected-(IDE1-Pin_28-Pad28): track 13.8 -> 0.00 mm
- net /~{Bus-Reset}: track 68.8 -> 64.8 mm
- net /~{Bus-ACK}: track 62.0 -> 63.4 mm
- net GND: vias 49 -> 97
