File: Hardware/PikaPC_Host/main_bus.kicad_sch (KiCad schematic)
At the start: 25 parts, among them J2 DIN41612_03x32_C_Split, J3 Conn_01x03, U15 74ABT2244, U2 ATF1508AS, U6 74ALVC164245, Y3 16M

Commit message: updates for gerber output
Connections:
- net ~{Bus-Reset} is gone; now on net ~{Bus-Reset}_R: R32.1
Changed lines of the file:
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@@
 	(wire
 		(pts
-			(xy 190.5 114.3) (xy 203.2 114.3)
+			(xy 187.96 114.3) (xy 203.2 114.3)
 		)
 		(stroke
@@
 	(wire
 		(pts
-			(xy 190.5 121.92) (xy 203.2 121.92)
+			(xy 187.96 121.92) (xy 203.2 121.92)
 		)
 		(stroke
@@
 	(wire
 		(pts
-			(xy 190.5 137.16) (xy 203.2 137.16)
+			(xy 187.96 137.16) (xy 203.2 137.16)
 		)
 		(stroke
@@
 	(wire
 		(pts
-			(xy 190.5 129.54) (xy 203.2 129.54)
+			(xy 187.96 129.54) (xy 203.2 129.54)
 		)
 		(stroke
@@
 	(wire
 		(pts
-			(xy 190.5 132.08) (xy 203.2 132.08)
+			(xy 187.96 132.08) (xy 203.2 132.08)
 		)
 		(stroke
@@
 	(wire
 		(pts
-			(xy 190.5 139.7) (xy 203.2 139.7)
+			(xy 187.96 139.7) (xy 203.2 139.7)
 		)
 		(stroke
@@
 	(wire
 		(pts
-			(xy 190.5 116.84) (xy 203.2 116.84)
+			(xy 187.96 116.84) (xy 203.2 116.84)
 		)
 		(stroke
@@
 	(wire
 		(pts
-			(xy 190.5 119.38) (xy 203.2 119.38)
+			(xy 187.96 119.38) (xy 203.2 119.38)
 		)
 		(stroke
@@
 	(wire
 		(pts
-			(xy 190.5 127) (xy 203.2 127)
+			(xy 187.96 127) (xy 203.2 127)
 		)
 		(stroke
@@
 	(wire
 		(pts
-			(xy 190.5 124.46) (xy 203.2 124.46)
+			(xy 187.96 124.46) (xy 203.2 124.46)
 		)
 		(stroke
@@
 	(wire
 		(pts
-			(xy 190.5 134.62) (xy 203.2 134.62)
+			(xy 187.96 134.62) (xy 203.2 134.62)
 		)
 		(stroke
@@
 	)
 	(label "~{Bus-IACK}"
-		(at 190.5 124.46 0)
+		(at 187.96 124.46 0)
 		(effects
 			(font
@@
 	)
 	(label "~{Bus-ACK}"
-		(at 190.5 129.54 0)
+		(at 187.96 129.54 0)
 		(effects
 			(font
@@
 	)
 	(label "~{Bus-IRQ0}"
-		(at 190.5 114.3 0)
+		(at 187.96 114.3 0)
 		(effects
 			(font
@@
 	)
 	(label "~{Bus-BRACK}"
-		(at 190.5 137.16 0)
+		(at 187.96 137.16 0)
 		(effects
 			(font
@@
 	)
 	(label "~{Bus-BURST}"
-		(at 190.5 127 0)
+		(at 187.96 127 0)
 		(effects
 			(font
@@
 	)
 	(label "~{Bus-GNT}"
-		(at 190.5 134.62 0)
+		(at 187.96 134.62 0)
 		(effects
 			(font
@@
 	)
 	(label "~{Bus-IRQ2}"
-		(at 190.5 119.38 0)
+		(at 187.96 119.38 0)
 		(effects
 			(font
@@
 	)
 	(label "~{Bus-BERR}"
-		(at 190.5 139.7 0)
+		(at 187.96 139.7 0)
 		(effects
 			(font
@@
 	)
 	(label "~{Bus-REQ}"
-		(at 190.5 132.08 0)
+		(at 187.96 132.08 0)
 		(effects
 			(font
@@
 		)
 	)
-	(label "~{Bus-Reset}"
-		(at 190.5 121.92 0)
+	(label "~{Bus-Reset}_R"
+		(at 187.96 121.92 0)
 		(effects
 			(font
@@
 	)
 	(label "~{Bus-IRQ1}"
-		(at 190.5 116.84 0)
+		(at 187.96 116.84 0)
 		(effects
 			(font
