File: Hardware/PikaPC_SRAM/PikaPC_SRAM.kicad_pcb (KiCad board)
At the start: 2 copper layers, 101.6 x 101.6 mm, 44 parts, among them J1 DIN41612_03x32_C_Split, J2 Conn_02x08_Odd_Even, Q1 PN2222A, U1 AS6C4008-55PCN, U10 74AHCT573, U11 AS6C4008-55PCN, U12 74FCT2245, U13 74FCT2245, U14 74FCT2245, U15 74FCT2245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

Commit message: updates for gerber output
Routing:
- net ~{Bus-BE2}: track 78.3 -> 72.2 mm
- net ~{Bus-BE3}: track 66.0 -> 64.1 mm
- net ~{Bus-Start}: track 135.3 -> 134.1 mm
- net GND: vias 299 -> 306
